File: eagle/NOMIDI_Controller_005_fix.brd (EAGLE design)
At the start: 198 x 210 mm, 134 parts, among them IC1 4067D, IC2 4067D, IC3 4067D, IC4 4067D, IC5 4067D, M0 SLIDEPOT-ALPS-60MM, M1 SLIDEPOT-ALPS-60MM, P0_0 US-EVUF3A, P0_1 US-EVUF3A, P0_2 US-EVUF3A, P0_3 US-EVUF3A, P0_4 US-EVUF3A, P0_5 US-EVUF3A, P0_6 US-EVUF3A, P0_7 US-EVUF3A, P0_8 US-EVUF3A, P0_9 US-EVUF3A, P1_0 US-EVUF3A, P1_1 US-EVUF3A, P1_2 US-EVUF3A, P1_3 US-EVUF3A, P1_4 US-EVUF3A, P1_5 US-EVUF3A, P1_6 US-EVUF3A, P1_7 US-EVUF3A, P1_8 US-EVUF3A, P1_9 US-EVUF3A, T1 BC547, T10 BC547, T2 BC547, T3 BC547, T4 BC547, T5 BC547, T6 BC547, T7 BC547, T8 BC547, T9 BC547

Commit message: pre STATE perfomance
Routing:
- net SWITCH2_X: track 0.00 -> 120.0 mm, vias 0 -> 12
- net LED9: track 82.4 -> 84.0 mm
- net ADDR_B: track 218.8 -> 218.1 mm
Changed lines of the file:
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@@
 <wire x1="142.24" y1="20.32" x2="141.0208" y2="19.05" width="0.4064" layer="1"/>
 <wire x1="141.0208" y1="19.05" x2="138.43" y2="19.05" width="0.4064" layer="1"/>
+<wire x1="161.33" y1="164.45" x2="177.84" y2="164.45" width="0" layer="19" extent="1-1"/>
 </signal>
 <signal name="+3V3">
@@
 <wire x1="168.91" y1="149.225" x2="168.91" y2="146.05" width="0.4064" layer="16"/>
 <wire x1="168.91" y1="146.05" x2="168.91" y2="140.335" width="0.4064" layer="16"/>
-<wire x1="168.91" y1="140.335" x2="157.48" y2="140.335" width="0.4064" layer="16"/>
-<wire x1="157.48" y1="140.335" x2="154.305" y2="136.525" width="0.4064" layer="16"/>
+<wire x1="168.91" y1="140.335" x2="158.115" y2="140.335" width="0.4064" layer="16"/>
+<wire x1="158.115" y1="140.335" x2="154.305" y2="136.525" width="0.4064" layer="16"/>
 <wire x1="154.305" y1="136.525" x2="143.51" y2="136.525" width="0.4064" layer="16"/>
 <wire x1="143.51" y1="136.525" x2="139.7" y2="140.335" width="0.4064" layer="16"/>
@@
 <via x="141.605" y="165.1" extent="1-16" drill="0.35"/>
 <wire x1="141.605" y1="165.1" x2="143.5608" y2="165.1" width="0.2" layer="1"/>
-<wire x1="168.91" y1="179.07" x2="177.165" y2="187.325" width="0.1524" layer="1"/>
+<wire x1="175.26" y1="185.42" x2="173.99" y2="185.42" width="0.1524" layer="1"/>
+<wire x1="175.26" y1="185.42" x2="177.165" y2="187.325" width="0.1524" layer="1"/>
+<wire x1="173.99" y1="185.42" x2="167.64" y2="179.07" width="0.1524" layer="1"/>
 <wire x1="141.605" y1="179.705" x2="156.21" y2="179.705" width="0.1524" layer="1"/>
 <wire x1="156.21" y1="179.705" x2="156.845" y2="179.07" width="0.1524" layer="1"/>
-<wire x1="156.845" y1="179.07" x2="168.91" y2="179.07" width="0.1524" layer="1"/>
+<wire x1="156.845" y1="179.07" x2="167.64" y2="179.07" width="0.1524" layer="1"/>
 <wire x1="143.5608" y1="165.1" x2="147.955" y2="165.1" width="0.1524" layer="1"/>
 <wire x1="147.955" y1="165.1" x2="148.59" y2="164.465" width="0.1524" layer="1"/>
@@
 <wire x1="141.605" y1="55.245" x2="141.605" y2="55.88" width="0.1524" layer="1"/>
 <wire x1="141.605" y1="55.88" x2="142.24" y2="56.515" width="0.1524" layer="1"/>
-<wire x1="142.24" y1="56.515" x2="145.415" y2="56.515" width="0.1524" layer="1"/>
+<wire x1="142.24" y1="56.515" x2="146.05" y2="56.515" width="0.1524" layer="1"/>
 <via x="146.05" y="92.075" extent="1-16" drill="0.35"/>
-<wire x1="146.05" y1="92.075" x2="146.05" y2="93.345" width="0.2" layer="16"/>
-<wire x1="146.05" y1="93.345" x2="146.05" y2="95.885" width="0.2" layer="16"/>
+<wire x1="146.05" y1="92.075" x2="146.05" y2="95.885" width="0.2" layer="16"/>
 <via x="146.05" y="95.885" extent="1-16" drill="0.35"/>
 <wire x1="146.05" y1="95.885" x2="146.05" y2="97.79" width="0.1524" layer="1"/>
 <wire x1="146.05" y1="97.79" x2="145.415" y2="98.425" width="0.1524" layer="1"/>
 <wire x1="145.415" y1="98.425" x2="143.5608" y2="98.425" width="0.1524" layer="1"/>
-<wire x1="145.415" y1="56.515" x2="146.05" y2="56.515" width="0.1524" layer="1"/>
 <wire x1="146.05" y1="56.515" x2="147.955" y2="58.42" width="0.1524" layer="1"/>
 <wire x1="147.955" y1="58.42" x2="147.955" y2="90.17" width="0.1524" layer="1"/>
 <wire x1="147.955" y1="90.17" x2="146.05" y2="92.075" width="0.1524" layer="1"/>
 <via x="147.955" y="180.34" extent="1-16" drill="0.35"/>
-<wire x1="168.91" y1="179.705" x2="156.845" y2="179.705" width="0.1524" layer="1"/>
+<wire x1="167.64" y1="179.705" x2="156.845" y2="179.705" width="0.1524" layer="1"/>
 <wire x1="156.845" y1="179.705" x2="156.21" y2="180.34" width="0.1524" layer="1"/>
 <wire x1="156.21" y1="180.34" x2="147.955" y2="180.34" width="0.1524" layer="1"/>
@@
 <wire x1="147.955" y1="165.735" x2="146.05" y2="163.83" width="0.2" layer="16"/>
 <via x="146.05" y="163.83" extent="1-16" drill="0.35"/>
-<wire x1="168.91" y1="179.705" x2="174.625" y2="185.42" width="0.1524" layer="1"/>
-<wire x1="174.625" y1="185.42" x2="174.625" y2="187.325" width="0.1524" layer="1"/>
+<wire x1="167.64" y1="179.705" x2="174.625" y2="186.69" width="0.1524" layer="1"/>
+<wire x1="174.625" y1="186.69" x2="174.625" y2="187.325" width="0.1524" layer="1"/>
 <wire x1="143.5608" y1="163.83" x2="146.05" y2="163.83" width="0.2" layer="1"/>
 <wire x1="146.05" y1="151.765" x2="148.59" y2="149.225" width="0.1524" layer="1"/>
@@
 <contactref element="IC5" pad="1"/>
 <contactref element="U$1" pad="18-A4/SDA0"/>
-<wire x1="164.465" y1="202.565" x2="143.5608" y2="111.125" width="0" layer="19" extent="1-1"/>
+<wire x1="143.5608" y1="111.125" x2="143.5608" y2="114.3508" width="0.1524" layer="1"/>
+<wire x1="143.5608" y1="114.3508" x2="144.78" y2="115.57" width="0.1524" layer="1"/>
+<wire x1="144.78" y1="115.57" x2="153.035" y2="115.57" width="0.1524" layer="1"/>
+<via x="153.035" y="115.57" extent="1-16" drill="0.35"/>
+<wire x1="153.035" y1="115.57" x2="153.035" y2="133.35" width="0.1524" layer="16"/>
+<wire x1="153.035" y1="133.35" x2="154.305" y2="134.62" width="0.1524" layer="16"/>
+<via x="154.305" y="134.62" extent="1-16" drill="0.35"/>
+<wire x1="154.305" y1="134.62" x2="154.305" y2="137.795" width="0.1524" layer="1"/>
+<via x="154.305" y="137.795" extent="1-16" drill="0.35"/>
+<wire x1="154.305" y1="137.795" x2="160.02" y2="143.51" width="0.1524" layer="16"/>
+<wire x1="160.02" y1="143.51" x2="166.37" y2="143.51" width="0.1524" layer="16"/>
+<via x="166.37" y="143.51" extent="1-16" drill="0.35"/>
+<wire x1="166.37" y1="143.51" x2="170.815" y2="143.51" width="0.1524" layer="1"/>
+<wire x1="170.815" y1="143.51" x2="171.45" y2="144.145" width="0.1524" layer="1"/>
+<wire x1="171.45" y1="144.145" x2="171.45" y2="157.48" width="0.1524" layer="1"/>
+<via x="171.45" y="157.48" extent="1-16" drill="0.35"/>
+<wire x1="171.45" y1="166.37" x2="171.45" y2="157.48" width="0.1524" layer="16"/>
+<via x="171.45" y="166.37" extent="1-16" drill="0.35"/>
+<wire x1="171.45" y1="166.37" x2="171.45" y2="173.99" width="0.1524" layer="1"/>
+<via x="171.45" y="173.99" extent="1-16" drill="0.35"/>
+<wire x1="171.45" y1="173.99" x2="171.45" y2="175.895" width="0.1524" layer="16"/>
+<via x="171.45" y="175.895" extent="1-16" drill="0.35"/>
+<wire x1="171.45" y1="175.895" x2="171.45" y2="181.61" width="0.1524" layer="1"/>
+<via x="172.72" y="182.88" extent="1-16" drill="0.35"/>
+<wire x1="171.45" y1="181.61" x2="172.72" y2="182.88" width="0.1524" layer="1"/>
+<wire x1="172.72" y1="182.88" x2="170.815" y2="184.785" width="0.1524" layer="16"/>
+<via x="170.815" y="184.785" extent="1-16" drill="0.35"/>
+<wire x1="170.815" y1="184.785" x2="170.815" y2="187.96" width="0.1524" layer="1"/>
+<wire x1="170.815" y1="187.96" x2="170.18" y2="188.595" width="0.1524" layer="1"/>
+<wire x1="170.18" y1="188.595" x2="167.005" y2="188.595" width="0.1524" layer="1"/>
+<wire x1="167.005" y1="188.595" x2="165.1" y2="190.5" width="0.1524" layer="1"/>
+<via x="165.1" y="190.5" extent="1-16" drill="0.35"/>
+<wire x1="165.1" y1="195.58" x2="164.465" y2="196.215" width="0.1524" layer="16"/>
+<via x="164.465" y="196.215" extent="1-16" drill="0.35"/>
+<wire x1="164.465" y1="196.215" x2="164.465" y2="202.565" width="0.1524" layer="1"/>
+<wire x1="165.1" y1="190.5" x2="165.1" y2="195.58" width="0.1524" layer="16"/>
 </signal>
 <signal name="SWITCH2_INH">
@@
 <wire x1="151.765" y1="100.33" x2="151.765" y2="134.62" width="0.1524" layer="16"/>
 <via x="151.765" y="134.62" extent="1-16" drill="0.35"/>
-<wire x1="151.765" y1="134.62" x2="151.765" y2="136.525" width="0.1524" layer="1"/>
-<wire x1="151.765" y1="136.525" x2="154.305" y2="139.065" width="0.1524" layer="1"/>
-<via x="154.305" y="139.065" extent="1-16" drill="0.35"/>
-<wire x1="154.305" y1="139.065" x2="159.385" y2="144.145" width="0.1524" layer="16"/>
-<wire x1="159.385" y1="144.145" x2="159.385" y2="149.225" width="0.1524" layer="16"/>
-<wire x1="159.385" y1="149.225" x2="159.385" y2="149.86" width="0.1524" layer="16"/>
+<wire x1="151.765" y1="134.62" x2="151.765" y2="137.16" width="0.1524" layer="1"/>
+<wire x1="151.765" y1="137.16" x2="153.035" y2="138.43" width="0.1524" layer="1"/>
+<via x="153.035" y="138.43" extent="1-16" drill="0.35"/>
+<wire x1="153.035" y1="138.43" x2="159.385" y2="144.78" width="0.1524" layer="16"/>
+<wire x1="159.385" y1="144.78" x2="159.385" y2="149.86" width="0.1524" layer="16"/>
 <wire x1="159.385" y1="149.86" x2="162.56" y2="153.035" width="0.1524" layer="16"/>
 <wire x1="162.56" y1="153.035" x2="162.56" y2="156.21" width="0.1524" layer="16"/>
@@
 <wire x1="160.655" y1="179.705" x2="160.655" y2="180.975" width="0.1524" layer="16"/>
 <wire x1="160.655" y1="180.975" x2="160.02" y2="181.61" width="0.1524" layer="16"/>
-<wire x1="160.02" y1="181.61" x2="159.385" y2="181.61" width="0.1524" layer="16"/>
-<wire x1="159.385" y1="181.61" x2="157.48" y2="181.61" width="0.1524" layer="16"/>
+<wire x1="160.02" y1="181.61" x2="157.48" y2="181.61" width="0.1524" layer="16"/>
 <wire x1="157.48" y1="181.61" x2="156.845" y2="182.88" width="0.1524" layer="16"/>
 <wire x1="156.845" y1="182.88" x2="158.75" y2="185.42" width="0.1524" layer="16"/>
@@
 <via x="157.48" y="194.945" extent="1-16" drill="0.35"/>
 <wire x1="157.48" y1="194.945" x2="159.385" y2="196.85" width="0.1524" layer="1"/>
-<wire x1="159.385" y1="196.85" x2="173.355" y2="196.85" width="0.1524" layer="1"/>
+<wire x1="159.385" y1="196.85" x2="162.56" y2="196.85" width="0.1524" layer="1"/>
+<wire x1="162.56" y1="196.85" x2="164.465" y2="194.945" width="0.1524" layer="1"/>
+<wire x1="164.465" y1="194.945" x2="167.005" y2="194.945" width="0.1524" layer="1"/>
+<wire x1="167.005" y1="194.945" x2="168.91" y2="196.85" width="0.1524" layer="1"/>
+<wire x1="168.91" y1="196.85" x2="173.355" y2="196.85" width="0.1524" layer="1"/>
 <via x="173.355" y="196.85" extent="1-16" drill="0.35"/>
 <wire x1="173.355" y1="196.85" x2="179.07" y2="196.85" width="0.1524" layer="16"/>

Commit message: bom link
Parts:
- R16, R17, R19, R20, R22, R23: value (none) -> 1 OHM
Changed lines of the file:
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@@
 <attribute name="VALUE" x="91.5162" y="131.191" size="1.27" layer="27" ratio="10" rot="R270"/>
 </element>
-<element name="R16" library="rcl" library_urn="urn:adsk.eagle:library:334" package="0207/7" package3d_urn="urn:adsk.eagle:package:23493/2" value="" x="7.62" y="165.1" smashed="yes" rot="R270">
+<element name="R16" library="rcl" library_urn="urn:adsk.eagle:library:334" package="0207/7" package3d_urn="urn:adsk.eagle:package:23493/2" value="1 OHM" x="7.62" y="165.1" smashed="yes" rot="R270">
 <attribute name="POPULARITY" value="46" x="7.62" y="165.1" size="1.778" layer="27" rot="R270" display="off"/>
 <attribute name="SPICEPREFIX" value="R" x="7.62" y="165.1" size="1.778" layer="27" rot="R270" display="off"/>
 <attribute name="VALUE" x="7.0612" y="167.386" size="1.27" layer="27" ratio="10" rot="R270"/>
 </element>
-<element name="R17" library="rcl" library_urn="urn:adsk.eagle:library:334" package="0207/7" package3d_urn="urn:adsk.eagle:package:23493/2" value="" x="12.7" y="199.39" smashed="yes" rot="R270">
+<element name="R17" library="rcl" library_urn="urn:adsk.eagle:library:334" package="0207/7" package3d_urn="urn:adsk.eagle:package:23493/2" value="1 OHM" x="12.7" y="199.39" smashed="yes" rot="R270">
 <attribute name="POPULARITY" value="46" x="12.7" y="199.39" size="1.778" layer="27" rot="R270" display="off"/>
 <attribute name="SPICEPREFIX" value="R" x="12.7" y="199.39" size="1.778" layer="27" rot="R270" display="off"/>
@@
 <attribute name="VALUE" x="10.414" y="117.5512" size="1.27" layer="27" ratio="10"/>
 </element>
-<element name="R19" library="rcl" library_urn="urn:adsk.eagle:library:334" package="0207/7" package3d_urn="urn:adsk.eagle:package:23493/2" value="" x="6.985" y="127.635" smashed="yes" rot="R270">
+<element name="R19" library="rcl" library_urn="urn:adsk.eagle:library:334" package="0207/7" package3d_urn="urn:adsk.eagle:package:23493/2" value="1 OHM" x="6.985" y="127.635" smashed="yes" rot="R270">
 <attribute name="POPULARITY" value="46" x="6.985" y="127.635" size="1.778" layer="27" rot="R270" display="off"/>
 <attribute name="SPICEPREFIX" value="R" x="6.985" y="127.635" size="1.778" layer="27" rot="R270" display="off"/>
 <attribute name="VALUE" x="6.4262" y="129.921" size="1.27" layer="27" ratio="10" rot="R270"/>
 </element>
-<element name="R20" library="rcl" library_urn="urn:adsk.eagle:library:334" package="0207/7" package3d_urn="urn:adsk.eagle:package:23493/2" value="" x="9.525" y="127.635" smashed="yes" rot="R270">
+<element name="R20" library="rcl" library_urn="urn:adsk.eagle:library:334" package="0207/7" package3d_urn="urn:adsk.eagle:package:23493/2" value="1 OHM" x="9.525" y="127.635" smashed="yes" rot="R270">
 <attribute name="POPULARITY" value="46" x="9.525" y="127.635" size="1.778" layer="27" rot="R270" display="off"/>
 <attribute name="SPICEPREFIX" value="R" x="9.525" y="127.635" size="1.778" layer="27" rot="R270" display="off"/>
@@
 <attribute name="VALUE" x="8.3312" y="156.591" size="1.27" layer="27" ratio="10" rot="R270"/>
 </element>
-<element name="R22" library="rcl" library_urn="urn:adsk.eagle:library:334" package="0207/7" package3d_urn="urn:adsk.eagle:package:23493/2" value="" x="10.16" y="144.145" smashed="yes" rot="R270">
+<element name="R22" library="rcl" library_urn="urn:adsk.eagle:library:334" package="0207/7" package3d_urn="urn:adsk.eagle:package:23493/2" value="1 OHM" x="10.16" y="144.145" smashed="yes" rot="R270">
 <attribute name="POPULARITY" value="46" x="10.16" y="144.145" size="1.778" layer="27" rot="R270" display="off"/>
 <attribute name="SPICEPREFIX" value="R" x="10.16" y="144.145" size="1.778" layer="27" rot="R270" display="off"/>
 <attribute name="VALUE" x="9.6012" y="146.431" size="1.27" layer="27" ratio="10" rot="R270"/>
 </element>
-<element name="R23" library="rcl" library_urn="urn:adsk.eagle:library:334" package="0207/7" package3d_urn="urn:adsk.eagle:package:23493/2" value="" x="15.24" y="115.57" smashed="yes">
+<element name="R23" library="rcl" library_urn="urn:adsk.eagle:library:334" package="0207/7" package3d_urn="urn:adsk.eagle:package:23493/2" value="1 OHM" x="15.24" y="115.57" smashed="yes">
 <attribute name="POPULARITY" value="46" x="15.24" y="115.57" size="1.778" layer="27" display="off"/>
 <attribute name="SPICEPREFIX" value="R" x="15.24" y="115.57" size="1.778" layer="27" display="off"/>
