File: pcb/NOMIDI_Controller_006_clean.brd (EAGLE design)
At the start: 198 x 210 mm, 134 parts, among them IC1 4067D, IC2 4067D, IC3 4067D, IC4 4067D, IC5 4067D, M0 SLIDEPOT-ALPS-60MM, M1 SLIDEPOT-ALPS-60MM, P0_0 US-EVUF3A, P0_1 US-EVUF3A, P0_2 US-EVUF3A, P0_3 US-EVUF3A, P0_4 US-EVUF3A, P0_5 US-EVUF3A, P0_6 US-EVUF3A, P0_7 US-EVUF3A, P0_8 US-EVUF3A, P0_9 US-EVUF3A, P1_0 US-EVUF3A, P1_1 US-EVUF3A, P1_2 US-EVUF3A, P1_3 US-EVUF3A, P1_4 US-EVUF3A, P1_5 US-EVUF3A, P1_6 US-EVUF3A, P1_7 US-EVUF3A, P1_8 US-EVUF3A, P1_9 US-EVUF3A, T1 BC817-16SMD, T10 BC817-16SMD, T2 BC817-16SMD, T3 BC817-16SMD, T4 BC817-16SMD, T5 BC817-16SMD, T6 BC817-16SMD, T7 BC817-16SMD, T8 BC817-16SMD, T9 BC817-16SMD

Commit message: update
Parts:
- R11, R12, R13, R14, R15, R24, R25, R26, R27, R28: value 4k7 -> 1k
Changed lines of the file:
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@@
 <attribute name="VALUE" x="88.265" y="119.38" size="1.27" layer="27" ratio="10" rot="R180"/>
 </element>
-<element name="R11" library="rcl" library_urn="urn:adsk.eagle:library:334" package="0207/7" package3d_urn="urn:adsk.eagle:package:23493/2" value="4k7" x="26.035" y="128.905" smashed="yes" rot="R270">
+<element name="R11" library="rcl" library_urn="urn:adsk.eagle:library:334" package="0207/7" package3d_urn="urn:adsk.eagle:package:23493/2" value="1k" x="26.035" y="128.905" smashed="yes" rot="R270">
 <attribute name="POPULARITY" value="46" x="26.035" y="128.905" size="1.778" layer="27" rot="R270" display="off"/>
 <attribute name="SPICEPREFIX" value="R" x="26.035" y="128.905" size="1.778" layer="27" rot="R270" display="off"/>
 <attribute name="VALUE" x="25.4762" y="131.191" size="1.27" layer="27" ratio="10" rot="R270"/>
 </element>
-<element name="R12" library="rcl" library_urn="urn:adsk.eagle:library:334" package="0207/7" package3d_urn="urn:adsk.eagle:package:23493/2" value="4k7" x="42.545" y="128.905" smashed="yes" rot="R270">
+<element name="R12" library="rcl" library_urn="urn:adsk.eagle:library:334" package="0207/7" package3d_urn="urn:adsk.eagle:package:23493/2" value="1k" x="42.545" y="128.905" smashed="yes" rot="R270">
 <attribute name="POPULARITY" value="46" x="42.545" y="128.905" size="1.778" layer="27" rot="R270" display="off"/>
 <attribute name="SPICEPREFIX" value="R" x="42.545" y="128.905" size="1.778" layer="27" rot="R270" display="off"/>
 <attribute name="VALUE" x="41.9862" y="131.191" size="1.27" layer="27" ratio="10" rot="R270"/>
 </element>
-<element name="R13" library="rcl" library_urn="urn:adsk.eagle:library:334" package="0207/7" package3d_urn="urn:adsk.eagle:package:23493/2" value="4k7" x="59.055" y="128.905" smashed="yes" rot="R270">
+<element name="R13" library="rcl" library_urn="urn:adsk.eagle:library:334" package="0207/7" package3d_urn="urn:adsk.eagle:package:23493/2" value="1k" x="59.055" y="128.905" smashed="yes" rot="R270">
 <attribute name="POPULARITY" value="46" x="59.055" y="128.905" size="1.778" layer="27" rot="R270" display="off"/>
 <attribute name="SPICEPREFIX" value="R" x="59.055" y="128.905" size="1.778" layer="27" rot="R270" display="off"/>
 <attribute name="VALUE" x="58.4962" y="131.191" size="1.27" layer="27" ratio="10" rot="R270"/>
 </element>
-<element name="R14" library="rcl" library_urn="urn:adsk.eagle:library:334" package="0207/7" package3d_urn="urn:adsk.eagle:package:23493/2" value="4k7" x="75.565" y="128.905" smashed="yes" rot="R270">
+<element name="R14" library="rcl" library_urn="urn:adsk.eagle:library:334" package="0207/7" package3d_urn="urn:adsk.eagle:package:23493/2" value="1k" x="75.565" y="128.905" smashed="yes" rot="R270">
 <attribute name="POPULARITY" value="46" x="75.565" y="128.905" size="1.778" layer="27" rot="R270" display="off"/>
 <attribute name="SPICEPREFIX" value="R" x="75.565" y="128.905" size="1.778" layer="27" rot="R270" display="off"/>
 <attribute name="VALUE" x="75.0062" y="131.191" size="1.27" layer="27" ratio="10" rot="R270"/>
 </element>
-<element name="R15" library="rcl" library_urn="urn:adsk.eagle:library:334" package="0207/7" package3d_urn="urn:adsk.eagle:package:23493/2" value="4k7" x="92.075" y="128.905" smashed="yes" rot="R270">
+<element name="R15" library="rcl" library_urn="urn:adsk.eagle:library:334" package="0207/7" package3d_urn="urn:adsk.eagle:package:23493/2" value="1k" x="92.075" y="128.905" smashed="yes" rot="R270">
 <attribute name="POPULARITY" value="46" x="92.075" y="128.905" size="1.778" layer="27" rot="R270" display="off"/>
 <attribute name="SPICEPREFIX" value="R" x="92.075" y="128.905" size="1.778" layer="27" rot="R270" display="off"/>
@@
 <attribute name="VALUE" x="184.785" y="119.38" size="1.27" layer="27" ratio="10" rot="R180"/>
 </element>
-<element name="R24" library="rcl" library_urn="urn:adsk.eagle:library:334" package="0207/7" package3d_urn="urn:adsk.eagle:package:23493/2" value="4k7" x="108.585" y="128.905" smashed="yes" rot="R270">
+<element name="R24" library="rcl" library_urn="urn:adsk.eagle:library:334" package="0207/7" package3d_urn="urn:adsk.eagle:package:23493/2" value="1k" x="108.585" y="128.905" smashed="yes" rot="R270">
 <attribute name="POPULARITY" value="46" x="130.175" y="207.645" size="1.778" layer="27" rot="R270" display="off"/>
 <attribute name="SPICEPREFIX" value="R" x="130.175" y="207.645" size="1.778" layer="27" rot="R270" display="off"/>
 <attribute name="VALUE" x="108.0262" y="131.191" size="1.27" layer="27" ratio="10" rot="R270"/>
 </element>
-<element name="R25" library="rcl" library_urn="urn:adsk.eagle:library:334" package="0207/7" package3d_urn="urn:adsk.eagle:package:23493/2" value="4k7" x="125.095" y="128.905" smashed="yes" rot="R270">
+<element name="R25" library="rcl" library_urn="urn:adsk.eagle:library:334" package="0207/7" package3d_urn="urn:adsk.eagle:package:23493/2" value="1k" x="125.095" y="128.905" smashed="yes" rot="R270">
 <attribute name="POPULARITY" value="46" x="142.24" y="217.17" size="1.778" layer="27" rot="R270" display="off"/>
 <attribute name="SPICEPREFIX" value="R" x="142.24" y="217.17" size="1.778" layer="27" rot="R270" display="off"/>
 <attribute name="VALUE" x="124.5362" y="131.191" size="1.27" layer="27" ratio="10" rot="R270"/>
 </element>
-<element name="R26" library="rcl" library_urn="urn:adsk.eagle:library:334" package="0207/7" package3d_urn="urn:adsk.eagle:package:23493/2" value="4k7" x="141.605" y="128.905" smashed="yes" rot="R270">
+<element name="R26" library="rcl" library_urn="urn:adsk.eagle:library:334" package="0207/7" package3d_urn="urn:adsk.eagle:package:23493/2" value="1k" x="141.605" y="128.905" smashed="yes" rot="R270">
 <attribute name="POPULARITY" value="46" x="154.305" y="226.695" size="1.778" layer="27" rot="R270" display="off"/>
 <attribute name="SPICEPREFIX" value="R" x="154.305" y="226.695" size="1.778" layer="27" rot="R270" display="off"/>
 <attribute name="VALUE" x="141.0462" y="131.191" size="1.27" layer="27" ratio="10" rot="R270"/>
 </element>
-<element name="R27" library="rcl" library_urn="urn:adsk.eagle:library:334" package="0207/7" package3d_urn="urn:adsk.eagle:package:23493/2" value="4k7" x="172.085" y="128.905" smashed="yes" rot="R270">
+<element name="R27" library="rcl" library_urn="urn:adsk.eagle:library:334" package="0207/7" package3d_urn="urn:adsk.eagle:package:23493/2" value="1k" x="172.085" y="128.905" smashed="yes" rot="R270">
 <attribute name="POPULARITY" value="46" x="185.42" y="195.58" size="1.778" layer="27" rot="R270" display="off"/>
 <attribute name="SPICEPREFIX" value="R" x="185.42" y="195.58" size="1.778" layer="27" rot="R270" display="off"/>
 <attribute name="VALUE" x="171.5262" y="131.191" size="1.27" layer="27" ratio="10" rot="R270"/>
 </element>
-<element name="R28" library="rcl" library_urn="urn:adsk.eagle:library:334" package="0207/7" package3d_urn="urn:adsk.eagle:package:23493/2" value="4k7" x="187.96" y="131.445" smashed="yes" rot="R270">
+<element name="R28" library="rcl" library_urn="urn:adsk.eagle:library:334" package="0207/7" package3d_urn="urn:adsk.eagle:package:23493/2" value="1k" x="187.96" y="131.445" smashed="yes" rot="R270">
 <attribute name="POPULARITY" value="46" x="196.85" y="207.645" size="1.778" layer="27" rot="R270" display="off"/>
 <attribute name="SPICEPREFIX" value="R" x="196.85" y="207.645" size="1.778" layer="27" rot="R270" display="off"/>
